Commit message: save

File: tracer_description/urdf/tracer.urdf (robot description, URDF)
Before this commit: robot omo_r1, 11 links, 10 joints
Links:
- removed link base_footprint
- removed link base_scan
- removed link camera_link
- removed link camera_rgb_frame
- removed link camera_rgb_optical_frame
- removed link caster_back_left_link
- removed link caster_back_right_link
- removed link imu_link
- removed link wheel_left_link
- removed link wheel_right_link
- added link camera_frame
- added link laser
- link base_link: mass 8.2573504 -> None; geometry 
Joints:
- removed joint base_joint
- removed joint camera_rgb_joint
- removed joint camera_rgb_optical_joint
- removed joint caster_back_left_joint
- removed joint caster_back_right_joint
- removed joint imu_joint
- removed joint scan_joint
- removed joint wheel_left_joint
- removed joint wheel_right_joint
- added joint laser_joint: type fixed, parent base_link, child laser, origin xyz=0.17 0 0.325 rpy=0.0 0.0 3.141592
- joint camera_joint: child camera_link -> camera_frame; origin xyz=0.07 0.0 0.63 rpy=0 0.7 0 -> xyz=0.20 0.0 0.305 rpy=-1.5708 0.0 -1.5708

File: tracer_description/urdf/tracer.urdf.xacro (robot description, xacro)
@@ -1,10 +1,10 @@
 <?xml version="1.0" ?>
-<robot name="omo_r1" xmlns:xacro="http://ros.org/wiki/xacro">
-  <xacro:include filename="$(find omo_r1_description)/urdf/common_properties.xacro"/>
-  <link name="camera_link"/>
+<robot name="tracer" xmlns:xacro="http://ros.org/wiki/xacro">
+  <xacro:include filename="$(find tracer_description)/urdf/common_properties.xacro"/>
+  <link name="camera_frame"/>
   <joint name="camera_joint" type="fixed">
-    <parent link="camera_link"/>
+    <parent link="camera_frame"/>
     <child link="base_link" />
-    <origin xyz="1.0 0.0 1.0" rpy="0 0 0.0"/>
+    <origin xyz="0.20 0.0 0.305" rpy="-1.5708 0.0 -1.5708"/>
   </joint>
   <link name="laser"/>
@@ -12,5 +12,5 @@
     <parent link="base_link"/>
     <child link="laser"/>
-    <origin xyz="0.06 0 0.230" rpy="3.141592 3.141592 0.0"/>
+    <origin xyz="0.17 0 0.325" rpy="0.0 0.0 0.0"/>
   </joint>
 </robot>
